File: kicad_pico_counter_new/allegro_pico_counter_new.kicad_sch (KiCad schematic)
At the start: 30 parts, among them J1 power, J10 Conn_01x01, J11 Conn_01x01, J12 Conn_01x01, J2 i2c, J3 display, J4 sensor, J5 Conn_Coaxial, J6 Conn_01x03, J7 ground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

Commit message: update kicad and gitignore
Parts:
- added J13, J14: Conn_01x01, Connector_PinHeader_2.54mm:PinHeader_1x01_P2.54mm_Vertical, symbol Connector_Generic:Conn_01x01
- added R9: R, Resistor_SMD:R_0805_2012Metric, symbol Device:R
- added SW4: SW_Push, Button_Switch_SMD:SW_SPST_CK_RS282G05A3, symbol Switch:SW_Push
Connections:
- net +3.3V: now also R9.1
- net GND: now also SW4.2
- net at R1.2, U3.11 (CMP1_OUT), U4.3 (1A): now also J14.1 (Pin_1)
- net at U4.2 (1Y), U5.3: now also J13.1 (Pin_1)
- net at U1.26 (GPIO20): now also R9.2, SW4.1
Other:
- moved on the sheet: J12, R6
