File: kicad_pico_counter_new/allegro_pico_counter_new.kicad_pcb (KiCad board)
At the start: 2 copper layers, 50.8 x 53.3 mm, 30 parts, among them J1 power, J10 Conn_01x01, J11 Conn_01x01, J12 Conn_01x01, J2 i2c, J3 display, J4 sensor, J5 Conn_Coaxial, J6 Conn_01x03, J7 ground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

Commit message: update kicad and gitignore
Parts:
- added J13: Conn_01x01, Connector_PinHeader_2.54mm:PinHeader_1x01_P2.54mm_Vertical, F.Cu at (148.3, 109.7)
- added J14: Conn_01x01, Connector_PinHeader_2.54mm:PinHeader_1x01_P2.54mm_Vertical, F.Cu at (165.6, 98.3)
- added R9: R, Resistor_SMD:R_0805_2012Metric, F.Cu at (138.9, 112.3)
- added SW4: SW_Push, Button_Switch_SMD:SW_SPST_CK_RS282G05A3, F.Cu at (156.0, 116.6)
- C2: value C -> 10nF
- C3: value C -> 3.3uF
Connections:
- U1 pad 26: unconnected-(U1-Pad26) -> Net-(U1-GPIO20)
Routing:
- net Net-(U1-GPIO20): track 0.00 -> 17.2 mm, vias 0 -> 1
- net +3.3V: track 111.1 -> 122.3 mm, vias 2 -> 3
- net GND: track 299.6 -> 290.6 mm
- net Net-(J14-Pin_1): track 18.0 -> 24.6 mm
- net +5V: track 83.3 -> 78.2 mm
- net Net-(J12-Pin_1): track 53.1 -> 56.4 mm
- net Net-(J13-Pin_1): track 32.8 -> 35.6 mm
- net Net-(J4-Pin_2): track 24.3 -> 22.8 mm
- net Net-(U1-RUN): track 20.6 -> 19.1 mm

Commit message: update callback code , and pcb layout
Parts:
- moved J8 0.47 mm to (120.7, 87.5)
Routing:
- net GND: track 290.6 -> 293.7 mm
Changed lines of the file:
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@@
   )
   (footprint "Connector_PinHeader_2.54mm:PinHeader_1x04_P2.54mm_Vertical" (layer "F.Cu")
-    (at 120.18 87.49)
+    (at 120.65 87.49)
     (descr "Through hole straight pin header, 1x04, 2.54mm pitch, single row")
     (tags "Through hole pin header THT 1x04 2.54mm single row")
@@
   (segment (start 164.465 78.11) (end 160.65 78.11) (width 0.3) (layer "F.Cu") (net 1))
   (segment (start 158.0915 96.8775) (end 159.258 96.8775) (width 0.6) (layer "F.Cu") (net 1))
-  (segment (start 155.702 123.698) (end 156.046 124.042) (width 1) (layer "F.Cu") (net 1))
   (segment (start 160.65 78.11) (end 157.607 81.153) (width 0.3) (layer "F.Cu") (net 1))
   (segment (start 165.354 87.884) (end 165.354 91.059) (width 0.6) (layer "F.Cu") (net 1))
@@
   (segment (start 156.21 98.745) (end 156.21 100.33) (width 0.3) (layer "F.Cu") (net 1))
   (segment (start 131.318 85.09) (end 136.398 85.09) (width 0.75) (layer "F.Cu") (net 1))
-  (segment (start 156.046 124.042) (end 156.046 125.476) (width 1) (layer "F.Cu") (net 1))
   (segment (start 154.94 97.475) (end 156.21 98.745) (width 0.3) (layer "F.Cu") (net 1))
   (segment (start 139.083 82.405) (end 142.575 82.405) (width 0.75) (layer "F.Cu") (net 1))
@@
   (segment (start 120.18 95.11) (end 124.79 95.11) (width 0.25) (layer "F.Cu") (net 1))
   (segment (start 153.416 108.018999) (end 153.484999 107.95) (width 0.6) (layer "F.Cu") (net 1))
+  (segment (start 156.046 120.576) (end 156.046 125.476) (width 1) (layer "F.Cu") (net 1))
   (segment (start 157.48 81.28) (end 157.48 82.206) (width 0.25) (layer "F.Cu") (net 1))
   (segment (start 155.575 93.345) (end 155.575 94.361) (width 0.6) (layer "F.Cu") (net 1))
@@
   (segment (start 148.971 120.015) (end 151.638 120.015) (width 0.6) (layer "F.Cu") (net 1))
   (segment (start 136.398 85.09) (end 139.083 82.405) (width 0.75) (layer "F.Cu") (net 1))
+  (segment (start 155.956 120.486) (end 156.046 120.576) (width 1) (layer "F.Cu") (net 1))
   (segment (start 160.02 101.6) (end 161.925 99.695) (width 0.6) (layer "F.Cu") (net 1))
   (segment (start 158.934998 101.6) (end 160.02 101.6) (width 0.3) (layer "F.Cu") (net 1))
