File: kicad_pico_counter_alt/allegro_pico_counter_alt.kicad_sch (KiCad schematic)
At the start: 36 parts, among them J1 power, J10 Conn_01x01, J11 Conn_01x01, J12 Conn_01x01, J13 Conn_01x01, J14 Conn_01x01, J15 jump, J16 jump, J2 i2c, J3 display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

Commit message: add new pcb and schematic version, and change a pin in the code
Parts:
- removed J14: Conn_01x01, Connector_PinHeader_2.54mm:PinHeader_1x01_P2.54mm_Vertical, symbol Connector_Generic:Conn_01x01
- removed U4: CD74HC4050M96, CD74HC4050M96:CD74HC4050M96, symbol CD74HC4050M96:CD74HC4050M96
- added J9: Conn_01x01, Connector_PinHeader_2.54mm:PinHeader_1x01_P2.54mm_Vertical, symbol Connector_Generic:Conn_01x01
- added SW5: SW_Push, Button_Switch_SMD:SW_SPST_CK_RS282G05A3, symbol Switch:SW_Push
- added U4: 74HC2G34GW, Package_TO_SOT_SMD:SOT-363_SC-70-6_Handsoldering, symbol z_proj_parts:74HC2G34GW
Connections:
- net +3.3V: now also U4.5 (Vcc)
- net GND: now also SW5.2, U4.2 (GND)
- net at J11.1 (Pin_1): now also U4.4 (2Y)
- net at R1.2, U3.11 (CMP1_OUT): now also J9.1 (Pin_1), U4.1 (1A)
- net at R3.2, U3.10 (CMP2_OUT): now also U4.3 (2A)
- net at J13.1 (Pin_1), U5.3: now also U4.6 (1Y)
- net at U1.24 (GPIO18): now also SW5.1
Other:
- moved on the sheet: J11
